Commit message: stray folders removal

File: Ros2BridgeTest/Assets/URDF/mycobot_description/urdf/mycobot_280_pi/mycobot_280_pi.urdf (robot description, URDF)
Before this commit: robot firefighter, 8 links, 7 joints
Links:
- link g_base: geometry collision mesh filename=G_base.dae; visual mesh filename=G_base.dae
- link joint1: geometry collision mesh filename=joint1_pi.dae; visual mesh filename=joint1_pi.dae
- link joint2: geometry collision mesh filename=joint2.dae; visual mesh filename=joint2.dae
- link joint3: geometry collision mesh filename=joint3.dae; visual mesh filename=joint3.dae
- link joint4: geometry collision mesh filename=joint4.dae; visual mesh filename=joint4.dae
- link joint5: geometry collision mesh filename=joint5.dae; visual mesh filename=joint5.dae
- link joint6: geometry collision mesh filename=joint6.dae; visual mesh filename=joint6.dae
- link joint6_flange: geometry collision mesh filename=joint7.dae; visual mesh filename=joint7.dae
