Commit message: clean mesh imported

File: Ros2BridgeTest/Assets/URDF/mycobot_320_pi/mycobot_320_pi_arm_gripper.urdf (robot description, URDF)
Before this commit: robot firefighter, 15 links, 14 joints
Joints:
- joint gripper_base_to_gripper_right3: limit lower=-0.3 upper=0.7 effort=1000.0 velocity=1.0 -> lower=0 upper=1 effort=1000.0 velocity=1.0
